File: eagle/TLF01/TLF01.brd (EAGLE design)
At the start: 94 x 71.1 mm, 54 parts, among them IC1 TL072P, J1 2SK170, T1 2SC1815, T10 2SC1815, T2 2SC1815, T3 2SC1815, T4 2SC1815, T5 2SC1815, T6 2SC1815, T7 2SC1815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

Commit message: Update: eagle files
Parts:
- moved C8 5.08 mm to (72.4, 33.0)
- moved C9 5.08 mm to (82.5, 33.0)
- moved R17 5.08 mm to (72.4, 27.9)
- moved R18 5.08 mm to (82.5, 27.9)
- moved LED1 5.08 mm to (74.9, 22.9)
- moved LED2 5.08 mm to (80.0, 22.9)
- moved JP5 2.54 mm to (78.7, 15.2)
- moved JP11 2.54 mm to (78.7, 5.08)
- moved C7 2.54 mm to (66.0, 40.6)
- moved JP3 2.54 mm to (64.8, 27.9)
Connections:
- net N$20: now also C7.-; no longer C7.+
- net N$22: now also C7.+; no longer C7.-

Commit message: Update eagle files
Parts:
- JP3: value Resonance 1k/A POT -> Resonance
- JP6: value Ictrl 50k/B POT -> Ictrl
- LED1: value PL+ Red -> Red
- LED2: value PL- Green -> Green
- moved R10 5.39 mm to (57.1, 53.3), turned to 180 degrees
- moved JP2 2.54 mm to (33.0, 6.35)
- moved JP6 2.54 mm to (49.5, 5.08)
- moved JP7 2.54 mm to (57.1, 5.08)
- moved JP1 2.54 mm to (11.4, 25.4)
- moved JP8 2.54 mm to (48.3, 20.3)
- moved JP9 2.54 mm to (11.4, 22.9)
- moved R12 2.54 mm to (49.5, 22.9)
- turned C7 to 90 degrees
- turned JP10 to 270 degrees
- turned JP4 to 270 degrees
- turned LED1 to 180 degrees
- turned R17 to 180 degrees
Connections:
- removed net N$26: LED1.A, R17.1
- new net N$1: LED1.K, R17.2
- net GND: now also R17.1; no longer LED1.K
- net V+: now also LED1.A; no longer R17.2
Routing:
- net GND: track 0.00 -> 239.6 mm
- net V+: track 0.00 -> 108.8 mm, vias 0 -> 2
- net V-: track 0.00 -> 93.2 mm
- net N$24: track 0.00 -> 45.7 mm
- net N$2: track 0.00 -> 40.2 mm, vias 0 -> 2
- net N$31: track 0.00 -> 39.2 mm
- net N$13: track 0.00 -> 33.6 mm
- net N$12: track 0.00 -> 33.6 mm
- net N$11: track 0.00 -> 25.4 mm
- net ICTRL: track 0.00 -> 25.4 mm
- net N$20: track 0.00 -> 23.9 mm
- net ICTRL_EXT: track 0.00 -> 20.3 mm
- net N$3: track 0.00 -> 20.3 mm, vias 0 -> 2
- net N$7: track 0.00 -> 15.2 mm
- net N$5: track 0.00 -> 15.2 mm
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