File: eagle/TLF01/TLF01.sch (EAGLE design)
At the start: 54 parts, among them IC1 TL072P, J1 2SK170, T1 2SC1815, T10 2SC1815, T2 2SC1815, T3 2SC1815, T4 2SC1815, T5 2SC1815, T6 2SC1815, T7 2SC1815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

Commit message: Update: eagle files
Connections:
- net N$20: now also C7.-; no longer C7.+
- net N$22: now also C7.+; no longer C7.-
Other:
- moved on the sheet: C7
Changed lines of the file:
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@@
 <instance part="R13" gate="G$1" x="134.62" y="144.78"/>
 <instance part="R11" gate="G$1" x="124.46" y="121.92" rot="R90"/>
-<instance part="C7" gate="G$1" x="144.78" y="106.68"/>
+<instance part="C7" gate="G$1" x="144.78" y="104.14" rot="R180"/>
 <instance part="JP1" gate="G$1" x="20.32" y="53.34" rot="MR0"/>
 <instance part="R14" gate="1" x="144.78" y="55.88" rot="MR0"/>
@@
 <wire x1="160.02" y1="132.08" x2="144.78" y2="132.08" width="0.1524" layer="91"/>
 <junction x="144.78" y="132.08"/>
-<pinref part="C7" gate="G$1" pin="+"/>
-<wire x1="144.78" y1="109.22" x2="144.78" y2="132.08" width="0.1524" layer="91"/>
 <pinref part="IC1" gate="B" pin="OUT"/>
 <wire x1="142.24" y1="132.08" x2="144.78" y2="132.08" width="0.1524" layer="91"/>
@@
 <wire x1="167.64" y1="132.08" x2="160.02" y2="132.08" width="0.1524" layer="91"/>
 <junction x="160.02" y="132.08"/>
+<pinref part="C7" gate="G$1" pin="-"/>
+<wire x1="144.78" y1="109.22" x2="144.78" y2="132.08" width="0.1524" layer="91"/>
 </segment>
 </net>
@@
 <net name="N$22" class="0">
 <segment>
-<pinref part="C7" gate="G$1" pin="-"/>
-<wire x1="144.78" y1="101.6" x2="144.78" y2="83.82" width="0.1524" layer="91"/>
 <pinref part="JP3" gate="G$1" pin="1"/>
 <wire x1="144.78" y1="83.82" x2="147.32" y2="83.82" width="0.1524" layer="91"/>
-</segment>
-</net>
+<pinref part="C7" gate="G$1" pin="+"/>
+<wire x1="144.78" y1="101.6" x2="144.78" y2="83.82" width="0.1524" layer="91"/>
+</segment>
+</net>

Commit message: Update eagle files
Parts:
- JP3: value Resonance 1k/A POT -> Resonance
- JP6: value Ictrl 50k/B POT -> Ictrl
- LED1: value PL+ Red -> Red
- LED2: value PL- Green -> Green
Connections:
- removed net N$26: LED1.A, R17.1
- new net N$1: LED1.C, R17.2
- net GND: now also R17.1; no longer LED1.C
- net V+: now also LED1.A; no longer R17.2
Other:
- note added: "R8はPinSocketで実装"
- moved on the sheet: LED1, R17
Changed lines of the file:
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@@
 <part name="JP4" library="pinhead" library_urn="urn:adsk.eagle:library:325" deviceset="PINHD-1X2" device="" package3d_urn="urn:adsk.eagle:package:22435/2" value="FilterOut"/>
 <part name="GND4" library="supply1" library_urn="urn:adsk.eagle:library:371" deviceset="GND" device=""/>
-<part name="JP3" library="pinhead" library_urn="urn:adsk.eagle:library:325" deviceset="PINHD-1X2" device="" package3d_urn="urn:adsk.eagle:package:22435/2" value="Resonance 1k/A POT"/>
+<part name="JP3" library="pinhead" library_urn="urn:adsk.eagle:library:325" deviceset="PINHD-1X2" device="" package3d_urn="urn:adsk.eagle:package:22435/2" value="Resonance"/>
 <part name="GND5" library="supply1" library_urn="urn:adsk.eagle:library:371" deviceset="GND" device=""/>
 <part name="GND1" library="supply1" library_urn="urn:adsk.eagle:library:371" deviceset="GND" device=""/>
@@
 <part name="J1" library="toshiba-jfet" deviceset="2SK170" device=""/>
 <part name="R15" library="rcl" library_urn="urn:adsk.eagle:library:334" deviceset="R-EU_" device="0207/7" package3d_urn="urn:adsk.eagle:package:23493/1" value="1k"/>
-<part name="JP6" library="pinhead" library_urn="urn:adsk.eagle:library:325" deviceset="PINHD-1X2" device="" package3d_urn="urn:adsk.eagle:package:22435/2" value="Ictrl 50k/B POT"/>
+<part name="JP6" library="pinhead" library_urn="urn:adsk.eagle:library:325" deviceset="PINHD-1X2" device="" package3d_urn="urn:adsk.eagle:package:22435/2" value="Ictrl"/>
 <part name="R16" library="rcl" library_urn="urn:adsk.eagle:library:334" deviceset="R-EU_" device="0207/7" package3d_urn="urn:adsk.eagle:package:23493/1" value="1k"/>
 <part name="JP8" library="pinhead" library_urn="urn:adsk.eagle:library:325" deviceset="PINHD-1X3" device="" package3d_urn="urn:adsk.eagle:package:22458/2" value="IctlSelect"/>
 <part name="JP7" library="pinhead" library_urn="urn:adsk.eagle:library:325" deviceset="PINHD-1X2" device="" package3d_urn="urn:adsk.eagle:package:22435/2" value="IctrlExt"/>
 <part name="GND7" library="supply1" library_urn="urn:adsk.eagle:library:371" deviceset="GND" device=""/>
-<part name="LED1" library="led" library_urn="urn:adsk.eagle:library:259" deviceset="LED" device="3MM" package3d_urn="urn:adsk.eagle:package:15797/1" value="PL+ Red"/>
-<part name="LED2" library="led" library_urn="urn:adsk.eagle:library:259" deviceset="LED" device="3MM" package3d_urn="urn:adsk.eagle:package:15797/1" value="PL- Green"/>
+<part name="LED1" library="led" library_urn="urn:adsk.eagle:library:259" deviceset="LED" device="3MM" package3d_urn="urn:adsk.eagle:package:15797/1" value="Red"/>
+<part name="LED2" library="led" library_urn="urn:adsk.eagle:library:259" deviceset="LED" device="3MM" package3d_urn="urn:adsk.eagle:package:15797/1" value="Green"/>
 <part name="R17" library="rcl" library_urn="urn:adsk.eagle:library:334" deviceset="R-EU_" device="0207/7" package3d_urn="urn:adsk.eagle:package:23493/1" value="1k"/>
 <part name="R18" library="rcl" library_urn="urn:adsk.eagle:library:334" deviceset="R-EU_" device="0207/7" package3d_urn="urn:adsk.eagle:package:23493/1" value="1k"/>
@@
 <wire x1="134.62" y1="165.1" x2="104.14" y2="165.1" width="0.1524" layer="97"/>
 <wire x1="104.14" y1="165.1" x2="96.52" y2="149.86" width="0.1524" layer="97"/>
+<text x="76.2" y="17.78" size="1.778" layer="91">R8はPinSocketで実装</text>
+<wire x1="99.06" y1="17.78" x2="76.2" y2="17.78" width="0.1524" layer="97"/>
+<wire x1="76.2" y1="17.78" x2="68.58" y2="25.4" width="0.1524" layer="97"/>
 </plain>
 <instances>
@@
 <instance part="JP7" gate="G$1" x="215.9" y="116.84"/>
 <instance part="GND7" gate="1" x="205.74" y="109.22"/>
-<instance part="LED1" gate="G$1" x="218.44" y="43.18"/>
+<instance part="LED1" gate="G$1" x="218.44" y="55.88"/>
 <instance part="LED2" gate="G$1" x="231.14" y="55.88" rot="MR0"/>
-<instance part="R17" gate="G$1" x="218.44" y="53.34" rot="R90"/>
+<instance part="R17" gate="G$1" x="218.44" y="43.18" rot="R90"/>
 <instance part="R18" gate="G$1" x="231.14" y="43.18" rot="R90"/>
 <instance part="GND8" gate="1" x="218.44" y="33.02"/>
@@
 </segment>
 <segment>
-<pinref part="LED1" gate="G$1" pin="C"/>
-<pinref part="GND8" gate="1" pin="GND"/>
-<wire x1="218.44" y1="38.1" x2="218.44" y2="35.56" width="0.1524" layer="91"/>
-</segment>
-<segment>
 <pinref part="J1" gate="G$1" pin="G"/>
 <wire x1="180.34" y1="68.58" x2="177.8" y2="68.58" width="0.1524" layer="91"/>
@@
 <wire x1="190.5" y1="33.02" x2="190.5" y2="35.56" width="0.1524" layer="91"/>
 <junction x="190.5" y="35.56"/>
+</segment>
+<segment>
+<pinref part="R17" gate="G$1" pin="1"/>
+<pinref part="GND8" gate="1" pin="GND"/>
+<wire x1="218.44" y1="38.1" x2="218.44" y2="35.56" width="0.1524" layer="91"/>
 </segment>
 </net>
@@
 <segment>
 <pinref part="P+3" gate="1" pin="V+"/>
-<pinref part="R17" gate="G$1" pin="2"/>
+<pinref part="LED1" gate="G$1" pin="A"/>
 <wire x1="218.44" y1="60.96" x2="218.44" y2="58.42" width="0.1524" layer="91"/>
 </segment>
@@
 </segment>
 </net>
-<net name="N$26" class="0">
-<segment>
-<pinref part="R17" gate="G$1" pin="1"/>
-<pinref part="LED1" gate="G$1" pin="A"/>
-<wire x1="218.44" y1="48.26" x2="218.44" y2="45.72" width="0.1524" layer="91"/>
-</segment>
-</net>
 <net name="N$29" class="0">
 <segment>
@@
 </segment>
 </net>
+<net name="N$1" class="0">
+<segment>
+<pinref part="LED1" gate="G$1" pin="C"/>
+<pinref part="R17" gate="G$1" pin="2"/>
+<wire x1="218.44" y1="50.8" x2="218.44" y2="48.26" width="0.1524" layer="91"/>
+</segment>
+</net>
