File: TLF01_Antilog/eagle/TLF01_Antilog_MM/AntilogMM.brd (EAGLE design)
At the start: 45.7 x 70.8 mm, 23 parts, among them P1 PWRIN, T1 2SA1015, T2 2SC1815

Commit message: Update: AntilogMM
Parts:
- added JP6: EXTPWR, pinhead:1X03
Connections:
- net +9V: now also JP6.1
- net -9V: now also JP6.3
- net GND: now also JP6.2
Routing:
- net +9V: track 56.5 -> 79.4 mm
- net GND: track 116.0 -> 133.7 mm
- net -9V: track 58.7 -> 66.3 mm
Changed lines of the file:
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@@
 <text x="7.62" y="7.62" size="2.54" layer="51" font="vector" rot="R90">AntiLog-MM</text>
 <text x="40.64" y="40.64" size="1.27" layer="51" font="vector" rot="R90">http://dad8893.blogspot.com/</text>
+<polygon width="0" layer="101" pour="hatch">
+<vertex x="16.51" y="38.1"/>
+<vertex x="16.51" y="45.72"/>
+<vertex x="19.05" y="45.72"/>
+<vertex x="19.05" y="38.1"/>
+</polygon>
 </plain>
 <attributes>
@@
 </element>
 <element name="T2" library="transistor" library_urn="urn:adsk.eagle:library:402" package="TO92-ECB" package3d_urn="urn:adsk.eagle:package:29929/2" value="2SC1815" x="25.4" y="60.96" rot="R270"/>
+<element name="JP6" library="pinhead" library_urn="urn:adsk.eagle:library:325" package="1X03" package3d_urn="urn:adsk.eagle:package:22458/2" value="EXTPWR" x="35.56" y="10.16" rot="R90"/>
 </elements>
 <signals>
@@
 <contactref element="R10" pad="1"/>
 <wire x1="27.94" y1="15.24" x2="27.9" y2="15.2" width="0.4064" layer="16"/>
-<wire x1="27.9" y1="15.2" x2="27.9" y2="7.62" width="0.4064" layer="16"/>
+<wire x1="27.9" y1="15.2" x2="27.9" y2="12.7" width="0.4064" layer="16"/>
+<wire x1="27.9" y1="12.7" x2="27.9" y2="7.62" width="0.4064" layer="16"/>
 <wire x1="30.48" y1="15.24" x2="30.44" y2="15.2" width="0.4064" layer="16"/>
 <wire x1="30.44" y1="15.2" x2="27.9" y2="15.2" width="0.4064" layer="16"/>
@@
 <wire x1="33.02" y1="22.86" x2="30.48" y2="25.4" width="0.4064" layer="16"/>
 <wire x1="30.48" y1="25.4" x2="27.94" y2="25.4" width="0.4064" layer="16"/>
+<contactref element="JP6" pad="3"/>
+<wire x1="35.56" y1="12.7" x2="27.9" y2="12.7" width="0.4064" layer="16"/>
 </signal>
 <signal name="+9V">
@@
 <wire x1="12.7" y1="33.02" x2="10.16" y2="33.02" width="0.4064" layer="16"/>
 <wire x1="15.24" y1="15.24" x2="17.78" y2="15.24" width="0.4064" layer="16"/>
+<contactref element="JP6" pad="1"/>
+<wire x1="35.56" y1="7.62" x2="35.56" y2="2.54" width="0.4064" layer="16"/>
+<wire x1="35.56" y1="2.54" x2="22.86" y2="2.54" width="0.4064" layer="16"/>
+<wire x1="22.86" y1="2.54" x2="22.86" y2="7.62" width="0.4064" layer="16"/>
 </signal>
 <signal name="GND">
@@
 <wire x1="25.4" y1="63.5" x2="25.4" y2="66.04" width="1.016" layer="16"/>
 <wire x1="30.48" y1="50.8" x2="30.48" y2="66.04" width="1.016" layer="16"/>
+<contactref element="JP6" pad="2"/>
+<wire x1="35.56" y1="10.16" x2="30.48" y2="10.16" width="1.016" layer="16"/>
+<wire x1="30.48" y1="10.16" x2="30.48" y2="5.08" width="1.016" layer="16"/>
+<wire x1="30.48" y1="5.08" x2="25.4" y2="5.08" width="1.016" layer="16"/>
+<wire x1="25.4" y1="5.08" x2="25.4" y2="7.62" width="1.016" layer="16"/>
 </signal>
 <signal name="N$7">
