File: TLF01_Antilog/eagle/TLF01_Antilog_MM/AntilogMM.sch (EAGLE design)
At the start: 23 parts, among them P1 PWRIN, T1 2SA1015, T2 2SC1815

Commit message: Update: AntilogMM
Parts:
- added JP6: EXTPWR, pinhead:PINHD-1X3
Connections:
- net +9V: now also JP6.1
- net -9V: now also JP6.3
- net GND: now also JP6.2
Other:
- note added: "R3はピンソケットで実装"
Changed lines of the file:
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@@
 <part name="JP5" library="pinhead" library_urn="urn:adsk.eagle:library:325" deviceset="PINHD-1X2" device="" package3d_urn="urn:adsk.eagle:package:22435/2" value="TP_GND"/>
 <part name="GND11" library="supply1" library_urn="urn:adsk.eagle:library:371" deviceset="GND" device=""/>
+<part name="JP6" library="pinhead" library_urn="urn:adsk.eagle:library:325" deviceset="PINHD-1X3" device="" package3d_urn="urn:adsk.eagle:package:22458/2" value="EXTPWR"/>
 </parts>
 <sheets>
@@
 <wire x1="86.36" y1="106.68" x2="106.68" y2="106.68" width="0.1524" layer="97"/>
 <wire x1="106.68" y1="106.68" x2="111.76" y2="96.52" width="0.1524" layer="97"/>
+<text x="86.36" y="106.68" size="1.778" layer="91">R4はピンソケットで実装</text>
+<text x="106.68" y="38.1" size="1.778" layer="91">R3はピンソケットで実装</text>
+<wire x1="129.54" y1="38.1" x2="106.68" y2="38.1" width="0.1524" layer="97"/>
+<wire x1="106.68" y1="38.1" x2="101.6" y2="45.72" width="0.1524" layer="97"/>
 </plain>
 <instances>
@@
 <instance part="JP5" gate="G$1" x="137.16" y="50.8" rot="MR0"/>
 <instance part="GND11" gate="1" x="144.78" y="43.18"/>
+<instance part="JP6" gate="A" x="63.5" y="134.62" rot="MR0"/>
 </instances>
 <busses>
@@
 <pinref part="SUPPLY2" gate="G$1" pin="-9V"/>
 <junction x="86.36" y="121.92"/>
+<pinref part="JP6" gate="A" pin="3"/>
+<wire x1="66.04" y1="132.08" x2="86.36" y2="132.08" width="0.1524" layer="91"/>
+<junction x="86.36" y="132.08"/>
 </segment>
 <segment>
@@
 <pinref part="SUPPLY1" gate="G$1" pin="+9V"/>
 <junction x="86.36" y="147.32"/>
+<pinref part="JP6" gate="A" pin="1"/>
+<wire x1="66.04" y1="137.16" x2="86.36" y2="137.16" width="0.1524" layer="91"/>
+<junction x="86.36" y="137.16"/>
 </segment>
 <segment>
@@
 <wire x1="93.98" y1="134.62" x2="104.14" y2="134.62" width="0.1524" layer="91"/>
 <wire x1="104.14" y1="134.62" x2="104.14" y2="132.08" width="0.1524" layer="91"/>
+<pinref part="JP6" gate="A" pin="2"/>
+<wire x1="66.04" y1="134.62" x2="86.36" y2="134.62" width="0.1524" layer="91"/>
+<junction x="86.36" y="134.62"/>
 </segment>
 <segment>
