File: TLF01_Antilog/Antilog_NPNO/eagle/Antilog-NPNO/Antilog-NPNO.brd (EAGLE design)
At the start: 71.1 x 45.7 mm, 30 parts, among them CN1 PWRIN, IC1 NJM4580, T1 2SC1815, T2 2SC1815

Commit message: Update: Antilog-NPNO board Design
Parts:
- moved R14 4.02 mm to (53.3, 16.5), turned to 270 degrees
- moved JP5 2.54 mm to (7.62, 6.35)
- moved JP4 2.54 mm to (54.6, 7.62), turned to 0 degrees
- moved R11 2.54 mm to (58.4, 26.7)
- turned C2 to 0 degrees
Routing:
- net GND: track 0.00 -> 221.2 mm
- net +12V: track 0.00 -> 72.2 mm
- net -12V: track 0.00 -> 38.2 mm, vias 0 -> 2
- net N$17: track 0.00 -> 27.9 mm, vias 0 -> 2
- net N$9: track 0.00 -> 27.9 mm
- net N$2: track 0.00 -> 20.3 mm
- net N$15: track 0.00 -> 12.7 mm
- net N$5: track 0.00 -> 7.62 mm
- net N$13: track 0.00 -> 5.08 mm
- net N$16: track 0.00 -> 5.08 mm
- net N$8: track 0.00 -> 2.54 mm
- net N$7: track 0.00 -> 2.54 mm
- net N$6: track 0.00 -> 2.54 mm
- net N$4: track 0.00 -> 2.54 mm
- net N$3: track 0.00 -> 2.54 mm
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Other:
- board text added: "Antilog-NPNO"
- board text added: "http://dad8893.blogspot.com/"
- board text added: "はピンソケットで実装"

Commit message: Add:テスト表
Parts:
- added JP6: TP_+12V, pinhead:1X01
Connections:
- net +12V: now also JP6.1
Routing:
- net +12V: track 72.2 -> 74.8 mm
Changed lines of the file:
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@@
 <layer number="97" name="Info" color="7" fill="1" visible="no" active="no"/>
 <layer number="98" name="Guide" color="6" fill="1" visible="no" active="no"/>
-<layer number="100" name="Grid" color="11" fill="1" visible="yes" active="yes"/>
+<layer number="100" name="Grid" color="11" fill="1" visible="no" active="yes"/>
 <layer number="101" name="Pinsocket" color="40" fill="1" visible="yes" active="yes"/>
 </layers>
@@
 <element name="T1" library="transistor-neu-to92" library_urn="urn:adsk.eagle:library:397" package="TO92-ECB" package3d_urn="urn:adsk.eagle:package:28756/2" value="2SC1815" x="53.34" y="30.48"/>
 <element name="T2" library="transistor-neu-to92" library_urn="urn:adsk.eagle:library:397" package="TO92-ECB" package3d_urn="urn:adsk.eagle:package:28756/2" value="2SC1815" x="53.34" y="22.86"/>
+<element name="JP6" library="pinhead" library_urn="urn:adsk.eagle:library:325" package="1X01" package3d_urn="urn:adsk.eagle:package:22485/2" value="TP_+12V" x="35.56" y="17.78"/>
 </elements>
 <signals>
@@
 <wire x1="33.02" y1="7.62" x2="40.64" y2="7.62" width="0.4064" layer="16"/>
 <wire x1="33.02" y1="12.7" x2="33.02" y2="7.62" width="0.4064" layer="16"/>
-<wire x1="33.02" y1="12.7" x2="33.02" y2="33.02" width="0.4064" layer="16"/>
+<wire x1="33.02" y1="12.7" x2="33.02" y2="17.78" width="0.4064" layer="16"/>
+<wire x1="33.02" y1="17.78" x2="33.02" y2="33.02" width="0.4064" layer="16"/>
 <wire x1="33.02" y1="33.02" x2="35.56" y2="33.02" width="0.4064" layer="16"/>
 <wire x1="35.56" y1="33.02" x2="35.56" y2="35.56" width="0.4064" layer="16"/>
@@
 <wire x1="30.48" y1="33.02" x2="33.02" y2="33.02" width="0.4064" layer="16"/>
 <wire x1="35.56" y1="35.56" x2="45.72" y2="35.56" width="0.4064" layer="16"/>
+<contactref element="JP6" pad="1"/>
+<wire x1="35.56" y1="17.78" x2="33.02" y2="17.78" width="0.4064" layer="16"/>
 </signal>
 <signal name="GND">
